File: KMKB-JP_SwitchPlate.kicad_pcb (KiCad board)
At the start: 2 copper layers, 285.4 x 94.9 mm, 198 parts

Commit message: 提出用のDXFをExport
Parts:
- moved K_L1 28.6 mm to (333.0, 396.4)
- moved K_:1 28.6 mm to (371.1, 396.4)
- moved K_;1 28.6 mm to (352.0, 396.4)
- moved K_A1 28.6 mm to (180.6, 396.4)
- moved K_CAPS1 28.6 mm to (154.4, 396.4)
- moved K_D1 28.6 mm to (218.7, 396.4)
- moved K_F1 28.6 mm to (237.7, 396.4)
- moved K_G1 28.6 mm to (256.8, 396.4)
- moved K_H1 28.6 mm to (275.8, 396.4)
- moved K_J1 28.6 mm to (294.9, 396.4)
- moved K_K1 28.6 mm to (313.9, 396.4)
- moved K_S1 28.6 mm to (199.6, 396.4)
- moved K_]1 28.6 mm to (390.1, 396.4)
- moved K_#2 28.6 mm to (185.3, 358.3)
- moved K_#6 28.6 mm to (261.5, 358.3)
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
Commit message: add plate name
Parts:
- moved K_[1 137.4 mm to (274.7, 51.3)
- moved K_#0_1 137.4 mm to (227.1, 32.2)
- moved K_#9 137.4 mm to (208.0, 32.2)
- moved K_,1 137.4 mm to (208.0, 89.4)
- moved K_.1 137.4 mm to (227.1, 89.4)
- moved K_@1 137.4 mm to (255.7, 51.3)
- moved K_C1 137.4 mm to (112.8, 89.4)
- moved K_HENK1 137.4 mm to (184.2, 108.4)
- moved K_J1 137.4 mm to (184.2, 70.3)
- moved K_K1 137.4 mm to (203.3, 70.3)
- moved K_LSPACE1 137.4 mm to (139.0, 108.4)
- moved K_TAB1 137.4 mm to (41.4, 51.3)
- moved K_U1 137.4 mm to (179.5, 51.3)
- moved K_WIN1 137.4 mm to (203.3, 108.4)
- moved K_X1 137.4 mm to (93.7, 89.4)
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Other:
- board text added: "OG60"
- board text added: "POKER互換"
- board text added: "TOFU60 2.0"
